File: cphp82001-pcb/cphp82001-pcb.kicad_pcb (KiCad board)
At the start: 2 copper layers, 56 x 44 mm, 34 parts, among them J1 USB_B_Micro, J2 PAD+, J3 PAD-, Q1 2N7002, U1 BQ21040, U2 TLV75801, U3 MAX40203AUK, U4 TPS3808DBV, U6 NCP360SNT

Commit message: Update rev3
Parts:
- removed D5: SM5817, Diode_SMD:D_SOD-123
- added C7: 1u, Capacitor_SMD:C_0805_2012Metric, F.Cu at (31.2, 7.80)
- added D4: PMEG40T10ERX, Diode_SMD:D_SOD-123, F.Cu at (30.3, 4.30)
- D1: value SM5817 -> PMEG40T10ERX
- R5: value 100k -> 97.6k
- R9: value 10k -> 33k
- moved REF** 2.00 mm to (51.1, 12.0)
- moved REF** 0.71 mm to (50.5, 37.0)
- moved R5 0.15 mm to (39.7, 2.95)
Routing:
- net /VCC: track 0.00 -> 11.0 mm
- net /VOUT: track 32.9 -> 35.5 mm
- net /EN: track 22.3 -> 20.9 mm
- net /GND: vias 30 -> 36

Commit message: Update board and render (v3.1)
Parts:
- removed F1: 500mA/24V, Fuse:Fuse_1210_3225Metric
- added G***: LOGO, LOGO, B.Cu at (48.0, 35.5)
- added REF**: graphic_batterysafety, george:graphic_batterysafety, B.Cu at (44.5, 25.5)
- R11: value 100k -> 1M
- R5: value 97.6k -> 95.3k
- moved REF** 44.0 mm to (6.50, 38.5)
- moved REF** 6.50 mm to (51.1, 5.50)
Connections:
- net Net-(U4-CT) renamed /BVCT
- net Net-(U4-SENSE) renamed /BSENSE
- J3 pad 1: /GNDF -> /GND
Routing:
- net /GNDF: track 46.8 -> 0.00 mm, vias 2 -> 0
- net /GND: track 1.02 -> 26.9 mm
Other:
- board text added: "CALCPSU"
- board text added: "MODEL: SERIAL: USB INPUT: PAD INPUT: PAD OUTPUT: BATTERY:"
- board text added: "github.com/calcpsu/cphp82001"
- board text removed: "CALCPSU.COM.AU"
- board text removed: "MODEL: SERIAL: USB INPUT: PAD INPUT: PAD OUTPUT: BATTERY: READ MANUAL BEFORE USING DO NOT SHORT CIRCUIT DO NOT BURN"

Commit message: A few more updates (v3.1)
Parts:
- moved C3 4.60 mm to (39.4, 7.80), turned to 0 degrees
- moved C7 4.60 mm to (35.8, 7.80)
- moved R5 4.30 mm to (35.5, 2.30), turned to 0 degrees
- moved D4 3.80 mm to (31.6, 7.85), turned to 0 degrees
- moved R4 3.73 mm to (34.5, 5.00), turned to 90 degrees
- moved R13 2.51 mm to (12.9, 8.00), turned to 0 degrees
- moved U3 2.20 mm to (31.4, 5.00), turned to 180 degrees
- moved U2 2.10 mm to (39.5, 5.00)
- moved C2 0.89 mm to (36.5, 5.00), turned to -90 degrees
- moved G*** 0.50 mm to (47.5, 35.5), turned to -90 degrees
- moved U6 0.40 mm to (9.10, 5.20)
- moved R9 0.27 mm to (9.36, 2.25)
Routing:
- net /GND: track 26.9 -> 14.5 mm, vias 36 -> 44
- net /VOUT: track 35.5 -> 30.7 mm
- net /EN: track 20.9 -> 16.2 mm
- net /VREG: track 10.2 -> 7.44 mm
- net /VCC: track 11.0 -> 12.0 mm
- net /BSENSE: track 6.69 -> 5.74 mm

Commit message: Rev3.2
Parts:
- removed C4: 1n, Capacitor_SMD:C_0805_2012Metric
- removed R10: 50k, Resistor_SMD:R_0805_2012Metric
- removed R6: 3M3, Resistor_SMD:R_0805_2012Metric
- removed R7: 500k, Resistor_SMD:R_0805_2012Metric
- removed U4: TPS3808DBV, george:SOT-23-6_TI_DBV6
- added U5: ~, Package_TO_SOT_SMD:SOT-23-3, F.Cu at (45.1, 3.80)
- moved R13 35.6 mm to (48.3, 3.80), turned to -90 degrees
- moved R11 4.72 mm to (45.4, 6.60)
- moved C5 0.40 mm to (48.3, 7.30)
- moved U1 0.34 mm to (19.0, 6.20)
Routing:
- net /B+: track 60.8 -> 54.6 mm
- net /BSENSE: track 5.74 -> 0.00 mm
- net /TS: track 45.4 -> 41.9 mm
- net /PROG2: track 16.1 -> 19.6 mm
- net /BVCT: track 1.67 -> 0.00 mm
- net /GND: vias 44 -> 50
Other:
- board text added: "BAT"

Commit message: rev3.3
Parts:
- removed D4: PMEG40T10ERX, Diode_SMD:D_SOD-123
- added Q2: AO3401A, Package_TO_SOT_SMD:SOT-23, F.Cu at (28.4, 4.06)
- added R3: 560k, Resistor_SMD:R_0805_2012Metric, F.Cu at (32.0, 2.30)
- added R6: 220k, Resistor_SMD:R_0805_2012Metric, F.Cu at (35.5, 2.30)
- added U7: MCP65R41T-120E/CHY, george:SOT-23-6_TI_DBV6, F.Cu at (32.0, 5.60)
- J1: value USB_B_Micro -> USB; footprint george:USB_ALIEX_4LEG -> mod_local:AMPHENOL_10118194-0001LF
- U5: value ~ -> APX803S-SA
- moved R2 14.1 mm to (12.0, 7.95), turned to 180 degrees
- moved D3 12.7 mm to (15.4, 7.95), turned to 180 degrees
- moved R13 8.20 mm to (52.9, 10.6), turned to 90 degrees
- moved C7 7.35 mm to (28.4, 7.60)
- moved R5 7.10 mm to (42.5, 2.30)
- moved R4 5.38 mm to (39.1, 2.30), turned to 0 degrees
- moved U3 4.62 mm to (35.9, 5.80)
- moved U2 3.35 mm to (42.9, 5.00)
- moved C2 3.30 mm to (39.8, 5.05)
- moved D2 2.68 mm to (24.8, 5.60), turned to -90 degrees
- moved J1 2.52 mm to (2.70, 5.15)
- moved U5 2.24 mm to (47.2, 2.90)
- moved R11 2.24 mm to (47.4, 5.70)
- moved R1 2.09 mm to (21.9, 3.81), turned to 90 degrees
- moved C3 1.30 mm to (40.6, 7.90), turned to 180 degrees
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Connections:
- D2 pad 1: /VCC -> /VOUT
Routing:
- net /VOUT: track 30.7 -> 51.3 mm, vias 1 -> 3
- net /VCC: track 12.0 -> 23.1 mm
- net /B+: track 54.6 -> 43.9 mm
- net /CHG: track 11.9 -> 6.50 mm, vias 0 -> 2
- net /PASSG: track 0.00 -> 4.48 mm
- net /VCOMP: track 0.00 -> 3.64 mm
- net /VREG: track 7.44 -> 10.7 mm
- net /TS: track 41.9 -> 45.0 mm
- net /PROG2: track 19.6 -> 16.9 mm
- net Net-(U7-+): track 0.00 -> 2.59 mm
- net /ADJ: track 5.46 -> 6.78 mm
- net /GND: track 14.5 -> 13.5 mm, vias 50 -> 44
- net /LCHG: track 2.56 -> 1.55 mm
- net /PROG: track 2.02 -> 2.75 mm
- net /VBUS1: track 8.01 -> 7.29 mm
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Other:
- outline, holes or cut-outs redrawn

Commit message: rev3.3a
Parts:
- removed R11: 1M, Resistor_SMD:R_0805_2012Metric
- removed R3: 560k, Resistor_SMD:R_0805_2012Metric
- removed R6: 220k, Resistor_SMD:R_0805_2012Metric
- removed U7: MCP65R41T-120E/CHY, george:SOT-23-6_TI_DBV6
- added U4: APX810-44SA, Package_TO_SOT_SMD:SOT-23-3, F.Cu at (31.9, 4.20)
- Q2: value AO3401A -> AO3413
- U5: value APX803S-SA -> APX809S-31SA
- moved R4 2.89 mm to (36.2, 2.30)
- moved R5 2.85 mm to (39.7, 2.30)
- moved C5 1.87 mm to (47.0, 6.00)
Connections:
- U3 pad 3: /EN -> unconnected-(U3-EN-Pad3)
Routing:
- net /EN: track 15.7 -> 1.95 mm, vias 2 -> 0
- net /VCOMP: track 3.64 -> 0.00 mm
- net /VOUT: track 51.3 -> 47.8 mm, vias 3 -> 1
- net /PASSG: track 4.48 -> 1.63 mm
- net Net-(U7-+): track 2.59 -> 0.00 mm
- net /VREG: track 10.7 -> 13.0 mm
- net /ADJ: track 6.78 -> 5.71 mm
