File: cphp82001-pcb/cphp82001-pcb.kicad_pcb (KiCad board)
At the start: 2 copper layers, 56 x 44 mm, 32 parts, among them J1 USB, J2 PAD+, J3 PAD-, Q1 2N7002, Q2 AO3413, U1 BQ21040, U2 TLV75801, U3 MAX40203AUK, U4 APX810-44SA, U5 APX809S-31SA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

Commit message: Update cphp82001-pcb.kicad_pcb
Parts:
- C7: value 1u -> 10u
- R1: value 1k3 -> 1k8
- R8: value 10k -> 11k
- moved R13 6.26 mm to (47.2, 8.00), turned to 0 degrees
- moved C5 0.27 mm to (47.2, 5.90)
Routing:
- net /GND: vias 44 -> 43

Commit message: rev3.5
Parts:
- removed C2: 1n, Capacitor_SMD:C_0805_2012Metric
- removed the REF** at (51.1, 5.50)
- added C4: 1u, Capacitor_SMD:C_0805_2012Metric, F.Cu at (33.6, 7.25)
- added G***: LOGO, LOGO, B.Cu at (52.1, 5.00)
- added JP1: NOREG, Resistor_SMD:R_0603_1608Metric, F.Cu at (36.7, 8.30)
- added JP2: NOLIM, Resistor_SMD:R_0603_1608Metric, F.Cu at (30.5, 5.40)
- added R3: 10k, Resistor_SMD:R_0805_2012Metric, F.Cu at (27.5, 7.29)
- added U7: NCP380HSN05, george:SOT-23-5_TI_DBV5, F.Cu at (30.5, 7.35)
- moved REF** 28.8 mm to (32.5, 26.0)
- moved Q2 6.33 mm to (34.6, 2.90), turned to 0 degrees
- moved R4 4.51 mm to (39.8, 5.01), turned to 90 degrees
- moved C7 3.92 mm to (27.5, 3.80), turned to -90 degrees
- moved R5 2.70 mm to (42.4, 2.20)
- moved C3 1.95 mm to (42.6, 7.90), turned to 0 degrees
- moved U4 1.87 mm to (30.6, 2.90), turned to 180 degrees
- moved U3 0.97 mm to (36.7, 6.35)
Connections:
- C7 pad 1: /VOUT -> /VOUTF
- D2 pad 1: /VOUT -> /VOUTF
- J2 pad 1: /VOUT -> /VOUTF
- U3 pad 3: unconnected-(U3-EN-Pad3) -> /EN
- U4 pad 3: /VOUT -> /VOUTF
Routing:
- net /VOUT: track 47.5 -> 0.00 mm, vias 1 -> 0
- net /VOUTF: track 0.00 -> 33.0 mm, vias 0 -> 1
- net /VREG: track 13.0 -> 0.00 mm
- net /EN: track 1.95 -> 12.0 mm, vias 0 -> 2
- net /VCC: track 23.1 -> 27.8 mm
- net /ADJ: track 5.71 -> 3.48 mm
- net Net-(U7-~{OC}): track 0.00 -> 1.62 mm
- net /TS: track 45.0 -> 44.2 mm
- net /GND: vias 43 -> 33
- added copper zone on F.Cu, net /VOUT
- added copper zone on F.Cu, net /VOUTF
- added copper zone on F.Cu, net /VREG
Other:
- board text added: "BATTERY LIPO 3.7V 10x34x50 2000mAh PROTECTED"
- board text added: "CPHP82001 V3.5 5V DC 400mA 50mA DC CC (16V MAX) 3.7V DC 400mA 3.7V 2000mAh LiPo"
- board text added: "MODEL: SERIAL: USB INPUT: PAD INPUT: PAD OUTPUT: CELL:"
- board text removed: "BATTERY LIPO 3.7V 10x34x50 2000mAh PROTECTED TYPE ONLY (DW01A+FS8205A OR SIMILAR)"
- board text removed: "CPHP82001 V3 5V DC 400mA 50mA DC CC (16V MAX) 3.7V DC 400mA 3.7V 2000mAh LiPo"
- board text removed: "MODEL: SERIAL: USB INPUT: PAD INPUT: PAD OUTPUT: BATTERY:"

Commit message: Rev 4.0
Parts:
- BT1: value LiPo -> Batt; footprint Connector_JST:JST_SH_BM03B-SRSS-TB_1x03-1MP_P1.00mm_Vertical -> george:JST_SH_BM03B-SRSS-TB_1x03-1MP_P1.00mm_Vertical_13PADS
- D1: value PMEG40T10ERX -> PMEG40T10ERX
- moved JP1 7.63 mm to (44.3, 7.60)
- moved C3 1.71 mm to (40.9, 8.05), turned to 180 degrees
- moved R13 0.40 mm to (47.6, 8.00)
- moved C5 0.35 mm to (47.5, 5.90)
Connections:
- JP1 pad 1: /VREG -> /B+
- JP1 pad 2: /VOUT -> /VREG
Routing:
- net /GND: track 13.5 -> 21.8 mm, vias 33 -> 32
- net /B+: track 44.3 -> 46.9 mm
- net /VREG: track 0.00 -> 1.71 mm
Other:
- board text added: "CPHP82001 V4.0 5V DC 400mA 50mA DC CC (16V MAX) 3.7V DC 400mA 3.7V 2000mAh LiPo"
- board text removed: "CPHP82001 V3.5 5V DC 400mA 50mA DC CC (16V MAX) 3.7V DC 400mA 3.7V 2000mAh LiPo"

Commit message: rev5
Parts:
- removed C3: 1u, Capacitor_SMD:C_0805_2012Metric
- removed JP1: NOREG, Resistor_SMD:R_0603_1608Metric
- removed JP2: NOLIM, Resistor_SMD:R_0603_1608Metric
- removed R3: 10k, Resistor_SMD:R_0805_2012Metric
- removed R4: 560k, Resistor_SMD:R_0805_2012Metric
- removed R5: 95.3k, Resistor_SMD:R_0805_2012Metric
- removed U2: TLV75801, george:SOT-23-5_TI_DBV5
- added D4: 1N4148W, Diode_SMD:D_SOD-123, F.Cu at (35.5, 3.40)
- R8: value 11k -> 9k1
- moved U3 6.23 mm to (42.9, 7.00)
- moved Q2 6.15 mm to (40.8, 3.25)
- moved C4 5.43 mm to (39.0, 7.00)
- moved C7 5.24 mm to (31.6, 7.00)
- moved U7 4.74 mm to (35.2, 7.00)
- moved C1 2.34 mm to (17.2, 3.20)
- moved D2 1.85 mm to (26.6, 5.60)
- moved U5 1.74 mm to (45.5, 2.90)
- moved R1 1.50 mm to (23.4, 3.81)
- moved R8 1.50 mm to (23.4, 7.30)
- moved Q1 1.20 mm to (14.2, 5.20)
- moved U1 1.07 mm to (20.1, 6.20)
- moved U6 0.79 mm to (9.71, 5.20)
- moved U4 0.35 mm to (30.6, 3.25)
- turned D3 to 0 degrees
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Connections:
- D3 pad 1: /CHG -> /LCHG
- D3 pad 2: /LCHG -> /VCC
- Q2 pad 3: /VCC -> Net-(D4-A)
- R2 pad 1: /LCHG -> /CHG
- R2 pad 2: /VCC -> /LCHG
- U3 pad 1: /VREG -> /B+
- U7 pad 3: Net-(U7-~{OC}) -> unconnected-(U7-~{OC}-Pad3)
Routing:
- net /VOUTF: track 33.0 -> 43.1 mm
- net /EN: track 12.0 -> 2.07 mm, vias 2 -> 0
- net /VOUT: track 0.00 -> 9.75 mm
- net /CHG: track 6.50 -> 14.8 mm
- net /PASSG: track 1.99 -> 8.13 mm
- net Net-(D4-A): track 0.00 -> 4.35 mm
- net /ADJ: track 3.48 -> 0.00 mm
- net /GND: track 21.8 -> 18.5 mm, vias 32 -> 24
- net /B+: track 46.9 -> 44.2 mm
- net /VREG: track 1.71 -> 0.00 mm
- net /PROG2: track 16.6 -> 14.9 mm
- net Net-(U7-~{OC}): track 1.62 -> 0.00 mm
- net /TS: track 44.2 -> 43.0 mm, vias 2 -> 0
- net /PROG: track 2.65 -> 3.48 mm
- net /VBUS1: track 7.29 -> 6.65 mm
- removed copper zone on F.Cu, net /VCC
- removed copper zone on F.Cu, net /VOUT
- removed copper zone on F.Cu, net /VOUTF
- removed copper zone on F.Cu, net /VREG
Other:
- board text added: "CPHP82001 V5.0 5V DC 400mA 50mA DC CC (16V MAX) 3.7V DC 400mA 3.7V 2000mAh (MAX) LiPo"
- board text removed: "CPHP82001 V4.0 5V DC 400mA 50mA DC CC (16V MAX) 3.7V DC 400mA 3.7V 2000mAh LiPo"
