File: cphp82001-pcb/cphp82001-pcb.kicad_sch (KiCad schematic)
At the start: 32 parts, among them J1 USB_B_Micro, J2 PAD+, J3 PAD-, Q1 2N7002, U1 BQ21040, U2 TLV75801, U3 MAX40203AUK, U4 TPS3808DBV, U6 NCP360SNT

Commit message: Update rev3
Parts:
- removed D5: SM5817, Diode_SMD:D_SOD-123, symbol Diode:1N5819
- added C7: 1u, Capacitor_SMD:C_0805_2012Metric, symbol Device:C
- added D4: PMEG40T10ERX, Diode_SMD:D_SOD-123, symbol Diode:1N5819
- D1: value SM5817 -> PMEG40T10ERX
- R5: value 100k -> 97.6k
- R9: value 10k -> 33k
Connections:
- net GND: now also C7.2
- net VCC: now also D4.1 (K)
- net VOUT: now also C7.1, D4.2 (A)
- net BSENSE: now reaches C4.1, R6.1, R7.2, U4.5 (SENSE)
- net BVCT: now reaches R10.1, U4.4 (CT)
Other:
- note added: "3.70V"
- note added: "40V 1A Vr ~ 3uA @ 5V/25C Vf 0.4V"
- note added: "5.0V (usb) 100mV (battery)"
- note added: "<-- 3uA"
- note added: "HP: <6.0V BAT: 3.7V"
- note added: "Iq=0.5uA"
- note added: "Iq=25uA"
- note added: "Iq=5uA"
- note added: "Iq=6uA"
- note added: "R5 OPTIONS: 100k0 --> 3.63V 97k6 --> 3.70V 95k3 --> 3.78V"
- note added: "RATED: --> 0 to 400mA (UNPLUGGED, ON) <-- 50mA (<16V) (PLUGGED IN)"
- note added: "RATED: 5.0V/400mA EN38.3 T.7: 10V/800mA"
- note added: "REV1 ADD Q1,R8,R9 REV1.1 U2=TPS73101, U4=S-8261ABJMD, R4=300k, R5=160k, update notes REV1.2 change D1 to 1N5817, change D2 to 5V6, R8=24k, Add C6 REV2 BOARD LAYOUT CHANGE REV3 ADD U6, C6, F1. change U4 to TPS3808 (+C4,R6,R7,R10,R11), change U1 to BQ21040, add Q2,D7,R13, move C2, add C7, new name"
- note added: "USB: 4.6V HP: <5.6V BAT: <V[B+]"
- note removed: "--> 80~125mA (UNPLUGGED, ON) <-- 50mA (<16V) (PLUGGED IN)"
- note removed: "0.5uA"
- note removed: "1mA typ"
- note removed: "25uA"
- note removed: "3.63V"
- note removed: "4.65V (USB) <5.1V (HP) <V[B+] (bat)"
- note removed: "6uA"
- note removed: "EN38.3 T.7: 10V/800mA"
- note removed: "REV1 ADD Q1,R8,R9 REV1.1 U2=TPS73101, U4=S-8261ABJMD, R4=300k, R5=160k, update notes REV1.2 change D1 to 1N5817, change D2 to 5V6, R8=24k, Add C6 REV2 BOARD LAYOUT CHANGE REV3 ADD U6, C6, F1. change U4 to TPS3808 (+C4,R6,R7,R10,R11), change U1 to BQ21040, add Q2,D7,R13, move C2"
- company: GR -> calcpsu.com.au
- moved on the sheet: BT1, C1, C2, C3, C4, C5, C6, D1, D2, D3, F1, J1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

Commit message: board layout update
Parts:
- R11: value 100k -> 1M
Changed lines of the file:
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@@
       (effects (font (size 1.27 1.27)) (justify right))
     )
-    (property "Value" "100k" (at 86.36 127 0)
+    (property "Value" "1M" (at 86.36 127 0)
       (effects (font (size 1.27 1.27)) (justify right))
     )

Commit message: Updates to model
Parts:
- R5: value 97.6k -> 100k
Changed lines of the file:
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@@
       (effects (font (size 1.27 1.27)) (justify left))
     )
-    (property "Value" "97.6k" (at 205.105 91.44 0)
+    (property "Value" "100k" (at 205.105 91.44 0)
       (effects (font (size 1.27 1.27)) (justify left))
     )

Commit message: Update board and render (v3.1)
Parts:
- removed F1: 500mA/24V, Fuse:Fuse_1210_3225Metric, symbol Device:Polyfuse
- R5: value 100k -> 95.3k
Connections:
- net GNDF is gone; now on net GND: J3.1 (Pin_1)
Other:
- note added: "Iq=25uA <400uA when on"
- note added: "REV1 ADD Q1,R8,R9 REV1.1 U2=TPS73101, U4=S-8261ABJMD, R4=300k, R5=160k, update notes REV1.2 change D1 to 1N5817, change D2 to 5V6, R8=24k, Add C6 REV2 BOARD LAYOUT CHANGE REV3 ADD U6, C6, F1. change U4 to TPS3808 (+C4,R6,R7,R10,R11), change U1 to BQ21040, add Q2,D7,R13, move C2, add C7, new name REV 3.1 remove F1, change R5 to 95.3k"
- note removed: "Iq=25uA"
- note removed: "REV1 ADD Q1,R8,R9 REV1.1 U2=TPS73101, U4=S-8261ABJMD, R4=300k, R5=160k, update notes REV1.2 change D1 to 1N5817, change D2 to 5V6, R8=24k, Add C6 REV2 BOARD LAYOUT CHANGE REV3 ADD U6, C6, F1. change U4 to TPS3808 (+C4,R6,R7,R10,R11), change U1 to BQ21040, add Q2,D7,R13, move C2, add C7, new name"
- moved on the sheet: J3
Changed lines of the file:
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@@
-    (stroke (width 0) (type default))
-  )
-  (wire (pts (xy 267.335 104.14) (xy 271.78 104.14))
     (stroke (width 0) (type default))
   )
@@
     (effects (font (size 1.27 1.27)) (justify left bottom))
   )
-  (text "Iq=25uA" (at 183.134 96.52 90)
+  (text "Iq=25uA\n<400uA when on" (at 182.88 99.06 90)
     (effects (font (size 1.27 1.27)) (justify left bottom))
   )
@@
     (effects (font (size 1.27 1.27)) (justify left bottom))
   )
-  (text "REV1 ADD Q1,R8,R9\n\nREV1.1 U2=TPS73101, U4=S-8261ABJMD, R4=300k, R5=160k, update notes\n\nREV1.2 change D1 to 1N5817, change D2 to 5V6, R8=24k, Add C6\n\nREV2 BOARD LAYOUT CHANGE\n\nREV3 ADD U6, C6, F1. change U4 to TPS3808 (+C4,R6,R7,R10,R11), change U1 to BQ21040, add Q2,D7,R13, move C2, add C7, new name"
+  (text "REV1 ADD Q1,R8,R9\n\nREV1.1 U2=TPS73101, U4=S-8261ABJMD, R4=300k, R5=160k, update notes\n\nREV1.2 change D1 to 1N5817, change D2 to 5V6, R8=24k, Add C6\n\nREV2 BOARD LAYOUT CHANGE\n\nREV3 ADD U6, C6, F1. change U4 to TPS3808 (+C4,R6,R7,R10,R11), change U1 to BQ21040, add Q2,D7,R13, move C2, add C7, new name\n\nREV 3.1 remove F1, change R5 to 95.3k"
     (at 17.78 194.31 0)
     (effects (font (size 1.27 1.27)) (justify left bottom))
@@
   )
   (label "TS" (at 102.235 132.08 180) (fields_autoplaced)
-    (effects (font (size 1.27 1.27)) (justify right bottom))
-  )
-  (label "GNDF" (at 270.51 104.14 270) (fields_autoplaced)
     (effects (font (size 1.27 1.27)) (justify right bottom))
   )
@@
     )
   )
-  (symbol (lib_id "Device:Polyfuse") (at 263.525 104.14 90) (unit 1)
-    (in_bom yes) (on_board yes) (dnp no) (fields_autoplaced)
-    (property "Reference" "F1" (at 263.525 97.79 90)
-      (effects (font (size 1.27 1.27)))
-    )
-    (property "Value" "500mA/24V" (at 263.525 100.33 90)
-      (effects (font (size 1.27 1.27)))
-    )
-    (property "Footprint" "Fuse:Fuse_1210_3225Metric" (at 268.605 102.87 0)
-      (effects (font (size 1.27 1.27)) (justify left) hide)
-    )
-    (property "Datasheet" "~" (at 263.525 104.14 0)
-      (effects (font (size 1.27 1.27)) hide)
-    )
-    (pin "1")
-    (pin "2")
-    (instances
-      (project "cphp82001-pcb"
-        (path "/e757784c-2761-4485-93b7-cc24857ba7f6"
-          (reference "F1") (unit 1)
-        )
-      )
-    )
-  )
   (symbol (lib_id "kicad_george:BQ21040") (at 140.335 72.39 0) (unit 1)
     (in_bom yes) (on_board yes) (dnp no) (fields_autoplaced)
@@
       (effects (font (size 1.27 1.27)) (justify left))
     )
-    (property "Value" "100k" (at 205.105 91.44 0)
+    (property "Value" "95.3k" (at 205.105 91.44 0)
       (effects (font (size 1.27 1.27)) (justify left))
     )
@@
     )
   )
-  (symbol (lib_id "Connector_Generic:Conn_01x01") (at 276.86 104.14 0) (unit 1)
+  (symbol (lib_id "Connector_Generic:Conn_01x01") (at 264.795 104.14 0) (unit 1)
     (in_bom yes) (on_board yes) (dnp no) (fields_autoplaced)
-    (property "Reference" "J3" (at 279.1951 102.8699 0)
-      (effects (font (size 1.27 1.27)) (justify left))
-    )
-    (property "Value" "PAD-" (at 279.1951 105.4099 0)
-      (effects (font (size 1.27 1.27)) (justify left))
-    )
-    (property "Footprint" "george:PAD_8x15" (at 276.86 104.14 0)
-      (effects (font (size 1.27 1.27)) hide)
-    )
-    (property "Datasheet" "~" (at 276.86 104.14 0)
-      (effects (font (size 1.27 1.27)) hide)
-    )
+    (property "Reference" "J3" (at 267.1301 102.8699 0)
+      (effects (font (size 1.27 1.27)) (justify left))
+    )
+    (property "Value" "PAD-" (at 267.1301 105.4099 0)
+      (effects (font (size 1.27 1.27)) (justify left))
+    )
+    (property "Footprint" "george:PAD_8x15" (at 264.795 104.14 0)
+      (effects (font (size 1.27 1.27)) hide)
+    )
+    (property "Datasheet" "~" (at 264.795 104.14 0)
+      (effects (font (size 1.27 1.27)) hide)
+    )

Commit message: Rev3.2
Parts:
- removed C4: 1n, Capacitor_SMD:C_0805_2012Metric, symbol Device:C
- removed R10: 50k, Resistor_SMD:R_0805_2012Metric, symbol Device:R
- removed R6: 3M3, Resistor_SMD:R_0805_2012Metric, symbol Device:R
- removed R7: 500k, Resistor_SMD:R_0805_2012Metric, symbol Device:R
- removed U4: TPS3808DBV, george:SOT-23-6_TI_DBV6, symbol Power_Supervisor:TPS3808DBV
- added U5: APX803S-SA, Package_TO_SOT_SMD:SOT-23-3, symbol kicad_george:APX803S-XXSA
Connections:
- net B+: now also U5.3 (VCC)
- net EN: now also U5.2 (~{RESET})
- net GND: now also U5.1 (GND)
- no-connect marks 5 -> 4
Other:
- note added: "REV1 ADD Q1,R8,R9 REV1.1 U2=TPS73101, U4=S-8261ABJMD, R4=300k, R5=160k, update notes REV1.2 change D1 to 1N5817, change D2 to 5V6, R8=24k, Add C6 REV2 BOARD LAYOUT CHANGE REV3 ADD U6, C6, F1. change U4 to TPS3808 (+C4,R6,R7,R10,R11), change U1 to BQ21040, add Q2,D7,R13, move C2, add C7, new name REV 3.1 remove F1, change R5 to 95.3k REV 3.2 change U5 to APX"
- note removed: "1uA"
- note removed: "REV1 ADD Q1,R8,R9 REV1.1 U2=TPS73101, U4=S-8261ABJMD, R4=300k, R5=160k, update notes REV1.2 change D1 to 1N5817, change D2 to 5V6, R8=24k, Add C6 REV2 BOARD LAYOUT CHANGE REV3 ADD U6, C6, F1. change U4 to TPS3808 (+C4,R6,R7,R10,R11), change U1 to BQ21040, add Q2,D7,R13, move C2, add C7, new name REV 3.1 remove F1, change R5 to 95.3k"

Commit message: rev3.3
Parts:
- removed D4: PMEG40T10ERX, Diode_SMD:D_SOD-123, symbol Diode:1N5819
- removed J1: USB_B_Micro, george:USB_ALIEX_4LEG, symbol Connector:USB_B_Micro
- added J1: USB, mod_local:AMPHENOL_10118194-0001LF, symbol amphenol_10118194:10118194-0001LF
- added Q2: AO3401A, Package_TO_SOT_SMD:SOT-23, symbol Transistor_FET:AO3401A
- added R3: 560k, Resistor_SMD:R_0805_2012Metric, symbol Device:R
- added R6: 220k, Resistor_SMD:R_0805_2012Metric, symbol Device:R
- added U7: MCP65R41T-120E/CHY, george:SOT-23-6_TI_DBV6, symbol Comparator:MCP65R41
Connections:
- net GND: now also J1.5, J1.S1 (SHIELD), J1.S2 (SHIELD__1), J1.S3 (SHIELD__2), J1.S4 (SHIELD__3), J1.S5 (SHIELD__4), J1.S6 (SHIELD__5), R6.2, U7.2 (V-)
- net VBUS1: now also J1.1
- net VCC: now also Q2.3 (D); no longer D2.1 (K)
- net VOUT: now also D2.1 (K), Q2.2 (S), R3.1, U7.6 (V+)
- new net: U7.3 (+), U7.5 (Vref)
- new net PASSG: Q2.1 (G), U7.1
- new net VCOMP: R3.2, R6.1, U7.4 (-)
Other:
- note added: "125uA (STBY, Vb<Vin)"
- note added: "3.5uA"
- note added: "3.78V"
- note added: "4.25V trigger"
- note added: "HP: <6.0V BAT: 3.78V USB: 4.2V (body diode Q2)"
- note added: "REV1 ADD Q1,R8,R9 REV1.1 U2=TPS73101, U4=S-8261ABJMD, R4=300k, R5=160k, update notes REV1.2 change D1 to 1N5817, change D2 to 5V6, R8=24k, Add C6 REV2 BOARD LAYOUT CHANGE REV3 ADD U6, C6, F1. change U4 to TPS3808 (+C4,R6,R7,R10,R11), change U1 to BQ21040, add Q2,D7,R13, move C2, add C7, new name REV 3.1 remove F1, change R5 to 95.3k REV 3.2 change U5 to APX REV 3.3 Add U7,R3,R6,Q2 for active back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"
- note removed: "3.70V"
- note removed: "HP: <6.0V BAT: 3.7V"
- note removed: "Iq=6uA"
- note removed: "REV1 ADD Q1,R8,R9 REV1.1 U2=TPS73101, U4=S-8261ABJMD, R4=300k, R5=160k, update notes REV1.2 change D1 to 1N5817, change D2 to 5V6, R8=24k, Add C6 REV2 BOARD LAYOUT CHANGE REV3 ADD U6, C6, F1. change U4 to TPS3808 (+C4,R6,R7,R10,R11), change U1 to BQ21040, add Q2,D7,R13, move C2, add C7, new name REV 3.1 remove F1, change R5 to 95.3k REV 3.2 change U5 to APX"
- moved on the sheet: BT1, C1, C2, C3, C5, C6, C7, D1, D2, D3, J2, J3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

Commit message: rev3.3a
Parts:
- removed R11: 1M, Resistor_SMD:R_0805_2012Metric, symbol Device:R
- removed R3: 560k, Resistor_SMD:R_0805_2012Metric, symbol Device:R
- removed R6: 220k, Resistor_SMD:R_0805_2012Metric, symbol Device:R
- removed U7: MCP65R41T-120E/CHY, george:SOT-23-6_TI_DBV6, symbol Comparator:MCP65R41
- added U4: APX810-44SA, Package_TO_SOT_SMD:SOT-23-3, symbol kicad_george:APX803S-XXSA
- Q2: value AO3401A -> AO3413
- U5: value APX803S-SA -> APX809S-31SA
Connections:
- net EN: no longer U3.3 (EN)
- net GND: now also U4.1 (GND)
- net PASSG: now also U4.2 (RESET)
- net VOUT: now also U4.3 (VCC)
- no-connect marks 4 -> 5
Other:
- note added: "3.1V trigger / 240ms timeout"
- note added: "4.4V trigger / 240ms timeout"
- note added: "REV1 ADD Q1,R8,R9 REV1.1 U2=TPS73101, U4=S-8261ABJMD, R4=300k, R5=160k, update notes REV1.2 change D1 to 1N5817, change D2 to 5V6, R8=24k, Add C6 REV2 BOARD LAYOUT CHANGE REV3 ADD U6, C6, F1. change U4 to TPS3808 (+C4,R6,R7,R10,R11), change U1 to BQ21040, add Q2,D7,R13, move C2, add C7, new name REV 3.1 remove F1, change R5 to 95.3k REV 3.2 change U5 to APX REV 3.3 Add U4,Q2 for active backfeed"
- note removed: "3.5uA"
- note removed: "4.25V trigger"
- note removed: "REV1 ADD Q1,R8,R9 REV1.1 U2=TPS73101, U4=S-8261ABJMD, R4=300k, R5=160k, update notes REV1.2 change D1 to 1N5817, change D2 to 5V6, R8=24k, Add C6 REV2 BOARD LAYOUT CHANGE REV3 ADD U6, C6, F1. change U4 to TPS3808 (+C4,R6,R7,R10,R11), change U1 to BQ21040, add Q2,D7,R13, move C2, add C7, new name REV 3.1 remove F1, change R5 to 95.3k REV 3.2 change U5 to APX REV 3.3 Add U7,R3,R6,Q2 for active back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"

Commit message: Minor update
Parts:
- C7: value 1u -> 10u
- R1: value 1k3 -> 1k8
- R8: value 10k -> 11k
Other:
- note added: "I_USB: 300mA I_HP: 48mA"
- note added: "Low battery lamp at 3.50V (3.60V for HP67)"
- note added: "REV1 ADD Q1,R8,R9 REV1.1 U2=TPS73101, U4=S-8261ABJMD, R4=300k, R5=160k, update notes REV1.2 change D1 to 1N5817, change D2 to 5V6, R8=24k, Add C6 REV2 BOARD LAYOUT CHANGE REV3 ADD U6, C6, F1. change U4 to TPS3808 (+C4,R6,R7,R10,R11), change U1 to BQ21040, add Q2,D7,R13, move C2, add C7, new name REV 3.1 remove F1, change R5 to 95.3k REV 3.2 change U5 to APX REV 3.3 Add U4,Q2 for active backfeed R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"
- note removed: "I_USB: 415mA I_HP: 48mA"
- note removed: "Low battery lamp at 3.50V"
- note removed: "R5 OPTIONS: 100k0 --> 3.63V 97k6 --> 3.70V 95k3 --> 3.78V"
- note removed: "REV1 ADD Q1,R8,R9 REV1.1 U2=TPS73101, U4=S-8261ABJMD, R4=300k, R5=160k, update notes REV1.2 change D1 to 1N5817, change D2 to 5V6, R8=24k, Add C6 REV2 BOARD LAYOUT CHANGE REV3 ADD U6, C6, F1. change U4 to TPS3808 (+C4,R6,R7,R10,R11), change U1 to BQ21040, add Q2,D7,R13, move C2, add C7, new name REV 3.1 remove F1, change R5 to 95.3k REV 3.2 change U5 to APX REV 3.3 Add U4,Q2 for active backfeed"
- note removed: "trip at 3.08V falling, 3.17V rising, +/- 1% 300ms delay"
Changed lines of the file:
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@@
     (effects (font (size 1.27 1.27)) (justify left bottom))
   )
-  (text "I_USB: 415mA\nI_HP: 48mA" (at 160.655 66.675 0)
+  (text "I_USB: 300mA\nI_HP: 48mA" (at 160.655 66.675 0)
     (effects (font (size 1.27 1.27)) (justify left bottom))
   )
@@
     (effects (font (size 1.27 1.27)) (justify left bottom))
   )
-  (text "R5 OPTIONS:\n100k0 --> 3.63V\n97k6 --> 3.70V\n95k3 --> 3.78V"
-    (at 200.025 113.665 0)
-    (effects (font (size 1.27 1.27)) (justify left bottom))
-  )
-  (text "trip at 3.08V falling, 3.17V rising, +/- 1%\n300ms delay"
-    (at 28.575 114.935 0)
-    (effects (font (size 1.27 1.27)) (justify left bottom))
-  )
   (text "5.5uA" (at 203.835 100.838 90)
     (effects (font (size 1.27 1.27)) (justify left bottom))
@@
     (effects (font (size 1.27 1.27)) (justify left bottom))
   )
-  (text "REV1 ADD Q1,R8,R9\n\nREV1.1 U2=TPS73101, U4=S-8261ABJMD, R4=300k, R5=160k, update notes\n\nREV1.2 change D1 to 1N5817, change D2 to 5V6, R8=24k, Add C6\n\nREV2 BOARD LAYOUT CHANGE\n\nREV3 ADD U6, C6, F1. change U4 to TPS3808 (+C4,R6,R7,R10,R11), change U1 to BQ21040, add Q2,D7,R13, move C2, add C7, new name\n\nREV 3.1 remove F1, change R5 to 95.3k\n\nREV 3.2 change U5 to APX\n\nREV 3.3 Add U4,Q2 for active backfeed"
+  (text "REV1 ADD Q1,R8,R9\n\nREV1.1 U2=TPS73101, U4=S-8261ABJMD, R4=300k, R5=160k, update notes\n\nREV1.2 change D1 to 1N5817, change D2 to 5V6, R8=24k, Add C6\n\nREV2 BOARD LAYOUT CHANGE\n\nREV3 ADD U6, C6, F1. change U4 to TPS3808 (+C4,R6,R7,R10,R11), change U1 to BQ21040, add Q2,D7,R13, move C2, add C7, new name\n\nREV 3.1 remove F1, change R5 to 95.3k\n\nREV 3.2 change U5 to APX\n\nREV 3.3 Add U4,Q2 for active backfeed\n\nREV 3.4 Change R1 to 1k8, R8 to 11k, C7 to 10u"
     (at 17.78 194.31 0)
     (effects (font (size 1.27 1.27)) (justify left bottom))
   )
-  (text "Low battery lamp at 3.50V" (at 28.575 109.855 0)
+  (text "Low battery lamp at 3.50V (3.60V for HP67)" (at 28.575 109.855 0)
     (effects (font (size 1.27 1.27)) (justify left bottom))
   )
@@
   (symbol (lib_id "Device:R") (at 116.205 81.28 180) (unit 1)
     (in_bom yes) (on_board yes) (dnp no) (fields_autoplaced)
-    (property "Reference" "R1" (at 118.745 80.01 0)
+    (property "Reference" "R1" (at 118.11 80.01 0)
       (effects (font (size 1.27 1.27)) (justify right))
     )
-    (property "Value" "1k3" (at 118.745 82.55 0)
+    (property "Value" "1k8" (at 118.11 82.55 0)
       (effects (font (size 1.27 1.27)) (justify right))
     )
@@
       (effects (font (size 1.27 1.27)) (justify left))
     )
-    (property "Value" "1u" (at 259.08 83.82 0)
+    (property "Value" "10u" (at 259.08 83.82 0)
       (effects (font (size 1.27 1.27)) (justify left))
     )
@@
   (symbol (lib_id "Device:R") (at 116.205 92.71 180) (unit 1)
     (in_bom yes) (on_board yes) (dnp no) (fields_autoplaced)
-    (property "Reference" "R8" (at 118.745 91.44 0)
+    (property "Reference" "R8" (at 118.11 91.44 0)
       (effects (font (size 1.27 1.27)) (justify right))
     )
-    (property "Value" "10k" (at 118.745 93.98 0)
+    (property "Value" "11k" (at 118.11 93.98 0)
       (effects (font (size 1.27 1.27)) (justify right))
     )
